File: board/board.kicad_pcb (KiCad board)
At the start: 2 copper layers, 21 x 13 mm, 1 part

Commit message: initial
Parts:
- added C1: 22uF, Capacitor_SMD:C_1206_3216Metric, F.Cu at (154.3, 95.3)
- added C2: 10pF, Capacitor_SMD:C_0603_1608Metric, F.Cu at (157.5, 99.5)
- added C3: 22uF, Capacitor_SMD:C_1206_3216Metric, F.Cu at (160.2, 98.8)
- added C4: 22uF, Capacitor_SMD:C_1206_3216Metric, F.Cu at (172.2, 98.8)
- added C5: 22uF, Capacitor_SMD:C_1206_3216Metric, F.Cu at (167.4, 98.8)
- added C6: 22uF, Capacitor_SMD:C_1206_3216Metric, F.Cu at (162.6, 98.8)
- added C7: 22uF, Capacitor_SMD:C_1206_3216Metric, F.Cu at (165.0, 98.8)
- added C8: 22uF, Capacitor_SMD:C_1206_3216Metric, F.Cu at (169.8, 98.8)
- added J1: 022_battery_cells, on_edge:on_edge_2x05_device, F.Cu at (140.0, 96.5)
- added J2: Conn_01x02_Male, Connector_PinHeader_2.54mm:PinHeader_1x02_P2.54mm_Vertical, F.Cu at (163.4, 91.9)
- added J3: 003_power, on_edge:on_edge_2x05_host, F.Cu at (185.0, 96.5)
- added L1: 470nH, b102:744383360047, F.Cu at (157.4, 93.6)
- added R1: 10k, Resistor_SMD:R_0603_1608Metric, F.Cu at (160.4, 93.2)
- added R2: 316k, Resistor_SMD:R_0603_1608Metric, F.Cu at (157.5, 101.0)
- added R3: 100k, Resistor_SMD:R_0603_1608Metric, F.Cu at (155.1, 100.3)
- added U1: TLV61220, Package_SON:WSON-8-1EP_2x2mm_P0.5mm_EP0.9x1.6mm, F.Cu at (157.6, 97.1)
- moved LOGO1 4.32 mm to (149.0, 94.8)
Routing:
- net GND: track 0.00 -> 41.6 mm, vias 0 -> 25
- net /step up/3.3V: track 0.00 -> 30.6 mm, vias 0 -> 16
- net /step up/in: track 0.00 -> 26.4 mm
- net /step up/SW: track 0.00 -> 8.61 mm
- net /step up/EN: track 0.00 -> 7.34 mm
- net /step up/FB: track 0.00 -> 4.87 mm
- added copper zone on B.Cu, net /step up/3.3V
- added copper zone on F.Cu, net /step up/3.3V
- added copper zone on F.Cu, net /step up/SW
- added copper zone on F.Cu, net /step up/in
- added copper zone on B.Cu, net GND
- added copper zone on F.Cu, net GND
Other:
- board size 21 x 13 mm -> 45 x 13 mm
- board text added: "enable"
- board text added: "osf.003"
- board text added: "osf.022"
- board text added: "osf.b102.v0.1"
